Commit message: update to project

File: src/arm_bot_description/urdf/arm_bot.xacro (robot description, xacro)
@@ -172,5 +172,5 @@
   <axis xyz="0.0 0.0 0.0"/>
 </joint>
-<joint name="Revolute 9" type="continuous">
+<joint name="Revolute_9" type="continuous">
   <origin xyz="0.0 0.0 0.04" rpy="0 0 0"/>
   <parent link="base_link"/>
@@ -178,5 +178,5 @@
   <axis xyz="0.0 0.0 1.0"/>
 </joint>
-<joint name="Revolute 10" type="continuous">
+<joint name="Revolute_10" type="continuous">
   <origin xyz="0.0 0.03 0.16" rpy="0 0 0"/>
   <parent link="link_1_1"/>
@@ -184,5 +184,5 @@
   <axis xyz="0.0 1.0 0.0"/>
 </joint>
-<joint name="Revolute 11" type="continuous">
+<joint name="Revolute_11" type="continuous">
   <origin xyz="-0.35 0.01 0.0" rpy="0 0 0"/>
   <parent link="link_2_1"/>
@@ -190,5 +190,5 @@
   <axis xyz="0.0 -1.0 0.0"/>
 </joint>
-<joint name="Revolute 12" type="continuous">
+<joint name="Revolute_12" type="continuous">
   <origin xyz="-0.3 -0.03 0.0" rpy="0 0 0"/>
   <parent link="link_3_1"/>
@@ -196,5 +196,5 @@
   <axis xyz="0.0 -1.0 0.0"/>
 </joint>
-<joint name="Revolute 13" type="continuous">
+<joint name="Revolute_13" type="continuous">
   <origin xyz="-0.06 -0.01 0.0" rpy="0 0 0"/>
   <parent link="link_4_1"/>
@@ -202,5 +202,5 @@
   <axis xyz="-1.0 0.0 0.0"/>
 </joint>
-<joint name="Slider 14" type="prismatic">
+<joint name="Slider_14" type="prismatic">
   <origin xyz="-0.045 0.05 0.0075" rpy="0 0 0"/>
   <parent link="link_5_1"/>
@@ -209,5 +209,5 @@
   <limit upper="0.0" lower="0.0" effort="100" velocity="100"/>
 </joint>
-<joint name="Slider 15" type="prismatic">
+<joint name="Slider_15" type="prismatic">
   <origin xyz="-0.045 -0.05 0.0075" rpy="0 0 0"/>
   <parent link="link_5_1"/>
